File: anotherworld/instruction_decoder.sch (KiCad schematic (older format))
At the start: 3 parts

Commit message: work in progress (stuff I've drawn in the couple past days)
Parts:
- added U?: 74LS138, ~, symbol 74LS138
- added U?: 74HC04, ~, symbol 74HC04
- added U? (x3): 74HC02, ~, symbol 74HC02
Connections:
- net GND: now also U?.7 (GND), U?.7 (GND), U?.7 (GND), U?.7 (GND), U?.8 (GND)
- net IR_4: now also U?.2; no longer U?.18 (E0), U?.19 (E1)
- net VCC: now also U?.14 (VCC), U?.14 (VCC), U?.14 (VCC), U?.14 (VCC), U?.16 (VCC)
- net at U?.18 (E0), U?.19 (E1): now also U?.1; no longer U?.2
- net ADD renamed -ADD
- net ADD_CONST renamed -ADD_CONST
- net AND renamed -AND
- net BLIT_FRAMEBUFFER renamed -BLIT_FRAMEBUFFER
- net BREAK renamed -BREAK
- net CALL renamed -CALL
- net CONDITIONAL_JUMP renamed -CONDITIONAL_JUMP
- net -CONDITIONAL_JUMP: now also U?.1, U?.4 (E1), U?.5 (E2)
- net COPY_VIDEO_PAGE renamed -COPY_VIDEO_PAGE
- net DJNZ renamed -DJNZ
- net FILL_VIDEO_PAGE renamed -FILL_VIDEO_PAGE
- net INVALID_OPCODE renamed -INVALID_OPCODE
- net JMP renamed -JMP
- net KILL_CHANNEL renamed -KILL_CHANNEL
- net LOAD_RESOURCE renamed -LOAD_RESOURCE
- net MOV renamed -MOV
- net MOV_CONST renamed -MOV_CONST
- net OR renamed -OR
- net PLAY_MUSIC renamed -PLAY_MUSIC
- net PLAY_SOUND renamed -PLAY_SOUND
- net RET renamed -RET
- net SELECT_VIDEO_PAGE renamed -SELECT_VIDEO_PAGE
- net SET_CHANNEL renamed -SET_CHANNEL
- net SET_PALETTE renamed -SET_PALETTE
- net SHL renamed -SHL
- net SHR renamed -SHR
- net SUB renamed -SUB
- net TEXT renamed -TEXT
- net UPDATE_CHANNEL renamed -UPDATE_CHANNEL
- new net: U?.1, U?.18 (E0), U?.19 (E1)
- new net: U?.2, U?.2
- new net: U?.2, U?.6 (E3)
- new net -INVALID_COND_JUMP: U?.7 (O7), U?.9 (O6)
- new net -JE: U?.15 (O0)
- new net -JG: U?.13 (O2)
- new net -JGE: U?.12 (O3)
- new net -JL: U?.11 (O4)
- new net -JLE: U?.10 (O5)
- new net -JNE: U?.14 (O1)
- new net -VIDEO: U?.1, U?.3, U?.3
- new net IR_6: U?.2
- new net IR_7: U?.3
- new net PARAM1_0: U?.1 (A0)
- new net PARAM1_1: U?.2 (A1)
- new net PARAM1_2: U?.3 (A2)
Other:
- moved on the sheet: U?, U?A
