File: anotherworld/alu.sch (KiCad schematic (older format))
At the start: 6 parts

Commit message: ALU circuitry
Parts:
- added P?: CONN_20, symbol CONN_20
- added U? (x4): 74LS374, ~, symbol 74LS374
Connections:
- net ALU_CARRY_IN: now also P?.12 (P12)
- net ALU_FUNCTION_0: now also P?.10 (P10)
- net ALU_FUNCTION_1: now also P?.9 (P9)
- net ALU_FUNCTION_2: now also P?.8 (P8)
- net ALU_FUNCTION_3: now also P?.7 (P7)
- net ALU_MODE: now also P?.11 (P11)
- net ALU_OUT_H: now also P?.5 (P5)
- net ALU_OUT_L: now also P?.6 (P6)
- net DATA_0: now also P?.20 (P20), U?.3 (D0), U?.3 (D0), U?.3 (D0), U?.3 (D0)
- net DATA_1: now also P?.19 (P19), U?.4 (D1), U?.4 (D1), U?.4 (D1), U?.4 (D1)
- net DATA_2: now also P?.18 (P18), U?.7 (D2), U?.7 (D2), U?.7 (D2), U?.7 (D2)
- net DATA_3: now also P?.17 (P17), U?.8 (D3), U?.8 (D3), U?.8 (D3), U?.8 (D3)
- net DATA_4: now also P?.16 (P16), U?.13 (D4), U?.13 (D4), U?.13 (D4), U?.13 (D4)
- net DATA_5: now also P?.15 (P15), U?.14 (D5), U?.14 (D5), U?.14 (D5), U?.14 (D5)
- net DATA_6: now also P?.14 (P14), U?.17 (D6), U?.17 (D6), U?.17 (D6), U?.17 (D6)
- net DATA_7: now also P?.13 (P13), U?.18 (D7), U?.18 (D7), U?.18 (D7), U?.18 (D7)
- net GND: now also U?.1 (OE), U?.1 (OE), U?.1 (OE), U?.1 (OE), U?.10 (GND), U?.10 (GND), U?.10 (GND), U?.10 (GND)
- net VCC: now also U?.20 (VCC), U?.20 (VCC), U?.20 (VCC), U?.20 (VCC)
- net ALU_A_0: no longer names the net of U?.2 (A0)
- net ALU_A_0: now also U?.2 (O0)
- net ALU_A_1: no longer names the net of U?.23 (A1)
- net ALU_A_1: now also U?.5 (O1)
- net ALU_A_10: no longer names the net of U?.21 (A2)
- net ALU_A_10: now also U?.6 (O2)
- net ALU_A_11: no longer names the net of U?.19 (A3)
- net ALU_A_11: now also U?.9 (O3)
- net ALU_A_12: no longer names the net of U?.2 (A0)
- net ALU_A_12: now also U?.12 (O4)
- net ALU_A_13: no longer names the net of U?.23 (A1)
- net ALU_A_13: now also U?.15 (O5)
- net ALU_A_14: no longer names the net of U?.21 (A2)
- net ALU_A_14: now also U?.16 (O6)
- net ALU_A_15: no longer names the net of U?.19 (A3)
- net ALU_A_15: now also U?.19 (O7)
- net ALU_A_2: no longer names the net of U?.21 (A2)
- net ALU_A_2: now also U?.6 (O2)
- net ALU_A_3: no longer names the net of U?.19 (A3)
- net ALU_A_3: now also U?.9 (O3)
- net ALU_A_4: no longer names the net of U?.2 (A0)
- net ALU_A_4: now also U?.12 (O4)
- net ALU_A_5: no longer names the net of U?.23 (A1)
- net ALU_A_5: now also U?.15 (O5)
- net ALU_A_6: no longer names the net of U?.21 (A2)
- net ALU_A_6: now also U?.16 (O6)
- net ALU_A_7: no longer names the net of U?.19 (A3)
- net ALU_A_7: now also U?.19 (O7)
- net ALU_A_8: no longer names the net of U?.2 (A0)
- net ALU_A_8: now also U?.2 (O0)
- net ALU_A_9: no longer names the net of U?.23 (A1)
- net ALU_A_9: now also U?.5 (O1)
- net ALU_B_0: no longer names the net of U?.1 (B0)
- net ALU_B_0: now also U?.2 (O0)
- net ALU_B_1: no longer names the net of U?.22 (B1)
- net ALU_B_1: now also U?.5 (O1)
- net ALU_B_10: no longer names the net of U?.20 (B2)
- net ALU_B_10: now also U?.6 (O2)
- net ALU_B_11: no longer names the net of U?.18 (B3)
- net ALU_B_11: now also U?.9 (O3)
- net ALU_B_12: no longer names the net of U?.1 (B0)
- net ALU_B_12: now also U?.12 (O4)
- net ALU_B_13: no longer names the net of U?.22 (B1)
- net ALU_B_13: now also U?.15 (O5)
- net ALU_B_14: no longer names the net of U?.20 (B2)
- net ALU_B_14: now also U?.16 (O6)
- net ALU_B_15: no longer names the net of U?.18 (B3)
- net ALU_B_15: now also U?.19 (O7)
- net ALU_B_2: no longer names the net of U?.20 (B2)
- net ALU_B_2: now also U?.6 (O2)
- net ALU_B_3: no longer names the net of U?.18 (B3)
- net ALU_B_3: now also U?.9 (O3)
- net ALU_B_4: no longer names the net of U?.1 (B0)
- net ALU_B_4: now also U?.12 (O4)
- net ALU_B_5: no longer names the net of U?.22 (B1)
- net ALU_B_5: now also U?.15 (O5)
- net ALU_B_6: no longer names the net of U?.20 (B2)
- net ALU_B_6: now also U?.16 (O6)
- net ALU_B_7: no longer names the net of U?.18 (B3)
- net ALU_B_7: now also U?.19 (O7)
- net ALU_B_8: no longer names the net of U?.1 (B0)
- net ALU_B_8: now also U?.2 (O0)
- net ALU_B_9: no longer names the net of U?.22 (B1)
- net ALU_B_9: now also U?.5 (O1)
- new net ALU_IN_AH_CLK: P?.3 (P3), U?.11 (Cp)
- new net ALU_IN_AL_CLK: P?.4 (P4), U?.11 (Cp)
- new net ALU_IN_BH_CLK: P?.1 (P1), U?.11 (Cp)
- new net ALU_IN_BL_CLK: P?.2 (P2), U?.11 (Cp)
Other:
- note added: "CONTROL SIGNALS"
- note added: "DATA BUS"
