File: anotherworld/alu.sch (KiCad schematic (older format))
At the start: 11 parts

Commit message: weekly workshop update
Other:
- note added: "ALU Input A High\nRegister"
- note added: "ALU Input A Low\nRegister"
- note added: "ALU Input B High\nRegister"
- note added: "ALU Input B Low\nRegister"
- note added: "ALU\nOutput\nHigh\nLatch"
- note added: "ALU\nOutput\nLow\nLatch"
Changed lines of the file:
@@
 LIBS:valves
 LIBS:27c801
+LIBS:o_ttl
 LIBS:anotherworld-cache
 EELAYER 27 0
@@
 $Descr A2 23386 16535
 encoding utf-8
-Sheet 6 8
+Sheet 5 7
 Title ""
 Date "9 aug 2016"
@@
 U 1 1 57A7AC01
 P 5200 5350
-F 0 "U?" H 5200 5350 60  0000 C CNN
-F 1 "74LS374" H 5250 5000 60  0000 C CNN
+F 0 "U?" H 5350 5100 60  0000 C CNN
+F 1 "74LS374" H 5250 4900 60  0000 C CNN
 F 2 "~" H 5200 5350 60  0000 C CNN
 F 3 "~" H 5200 5350 60  0000 C CNN
@@
 U 1 1 57A7B105
 P 6450 5350
-F 0 "U?" H 6450 5350 60  0000 C CNN
-F 1 "74LS374" H 6500 5000 60  0000 C CNN
+F 0 "U?" H 6600 5100 60  0000 C CNN
+F 1 "74LS374" H 6500 4900 60  0000 C CNN
 F 2 "~" H 6450 5350 60  0000 C CNN
 F 3 "~" H 6450 5350 60  0000 C CNN
@@
 U 1 1 57A7B6CE
 P 7850 4300
-F 0 "U?" H 7850 4300 60  0000 C CNN
-F 1 "74LS374" H 7900 3950 60  0000 C CNN
+F 0 "U?" H 8000 4050 60  0000 C CNN
+F 1 "74LS374" H 7900 3850 60  0000 C CNN
 F 2 "~" H 7850 4300 60  0000 C CNN
 F 3 "~" H 7850 4300 60  0000 C CNN
@@
 U 1 1 57A7B6E0
 P 9100 4300
-F 0 "U?" H 9100 4300 60  0000 C CNN
-F 1 "74LS374" H 9150 3950 60  0000 C CNN
+F 0 "U?" H 9250 4050 60  0000 C CNN
+F 1 "74LS374" H 9150 3850 60  0000 C CNN
 F 2 "~" H 9100 4300 60  0000 C CNN
 F 3 "~" H 9100 4300 60  0000 C CNN
@@
 Text Notes 20100 5450 0    118  ~ 0
 DATA BUS
+Text Notes 4850 5250 0    60   ~ 12
+ALU Input A Low\nRegister
+Text Notes 6100 5250 0    60   ~ 12
+ALU Input A High\nRegister
+Text Notes 7500 4200 0    60   ~ 12
+ALU Input B Low\nRegister
+Text Notes 8750 4200 0    60   ~ 12
+ALU Input B High\nRegister
+Text Notes 16850 11600 0    60   ~ 12
+ALU\nOutput\nLow\nLatch
+Text Notes 16850 13100 0    60   ~ 12
+ALU\nOutput\nHigh\nLatch
 $EndSCHEMATC
