File: anotherworld/alu.sch (KiCad schematic (older format))
At the start: 11 parts

Commit message: rescue (loading the project on a newer git-revision of kicad)
Parts:
- U? (x4): symbol 74LS181 -> 74LS181-RESCUE-anotherworld
- U? (x2): symbol 74LS245 -> 74LS245-RESCUE-anotherworld
- U? (x4): symbol 74LS374 -> 74LS374-RESCUE-anotherworld
Changed lines of the file:
@@
 EESchema Schematic File Version 2
-LIBS:power
-LIBS:device
-LIBS:transistors
-LIBS:conn
-LIBS:linear
-LIBS:regul
-LIBS:74xx
-LIBS:cmos4000
-LIBS:adc-dac
-LIBS:memory
-LIBS:xilinx
-LIBS:special
-LIBS:microcontrollers
-LIBS:dsp
-LIBS:microchip
-LIBS:analog_switches
-LIBS:motorola
-LIBS:texas
-LIBS:intel
-LIBS:audio
-LIBS:interface
-LIBS:digital-audio
-LIBS:philips
-LIBS:display
-LIBS:cypress
-LIBS:siliconi
-LIBS:opto
-LIBS:atmel
-LIBS:contrib
-LIBS:valves
+LIBS:anotherworld-rescue
 LIBS:27c801
 LIBS:o_ttl
 LIBS:jamma_connector
 LIBS:anotherworld-cache
-EELAYER 25 0
+EELAYER 26 0
 EELAYER END
 $Descr A2 23386 16535
@@
 $EndDescr
 $Comp
-L 74LS181 U?
+L 74LS181-RESCUE-anotherworld U?
 U 1 1 57A4B525
 P 8800 10250
@@
 $EndComp
 $Comp
-L 74LS181 U?
+L 74LS181-RESCUE-anotherworld U?
 U 1 1 57A4B896
 P 11000 10250
@@
 $EndComp
 $Comp
-L 74LS181 U?
+L 74LS181-RESCUE-anotherworld U?
 U 1 1 57A4B8B0
 P 13200 10250
@@
 $EndComp
 $Comp
-L 74LS181 U?
+L 74LS181-RESCUE-anotherworld U?
 U 1 1 57A4B8B6
 P 15400 10250
@@
 ALU_CARRY_IN
 $Comp
-L 74LS245 U?
+L 74LS245-RESCUE-anotherworld U?
 U 1 1 57A4E7D3
 P 17000 12050
@@
 $EndComp
 $Comp
-L 74LS245 U?
+L 74LS245-RESCUE-anotherworld U?
 U 1 1 57A4E7E0
 P 17000 13550
@@
 $EndComp
 $Comp
-L 74LS374 U?
+L 74LS374-RESCUE-anotherworld U?
 U 1 1 57A7AC01
 P 5200 5350
@@
 $EndComp
 $Comp
-L 74LS374 U?
+L 74LS374-RESCUE-anotherworld U?
 U 1 1 57A7B105
 P 6450 5350
@@
 $EndComp
 $Comp
-L 74LS374 U?
+L 74LS374-RESCUE-anotherworld U?
 U 1 1 57A7B6CE
 P 7850 4300
@@
 $EndComp
 $Comp
-L 74LS374 U?
+L 74LS374-RESCUE-anotherworld U?
 U 1 1 57A7B6E0
 P 9100 4300
