File: anotherworld/microcode.sch (KiCad schematic (older format))
At the start: 3 parts

Commit message: uCode ROM signals
Parts:
- added U? (x2): 27C512, symbol 27C512
- added U? (x2): 74HC04, ~, symbol 74HC04
- added U?: 74LS138, ~, symbol 74LS138
Connections:
- net ALU_OUT_H: now also U?.2
- net ALU_OUT_L: now also U?.2
- net CODEBANK_CLK: now also U?.13 (D2)
- net GND: now also U?.14 (GND), U?.14 (GND), U?.20 (CE), U?.20 (CE), U?.22 (OE), U?.22 (OE), U?.4 (E1), U?.5 (E2), U?.7 (GND), U?.7 (GND), U?.8 (GND)
- net IPH_CLK: now also U?.16 (D4)
- net IPL_CLK: now also U?.15 (D3)
- net OPCODE_CLK: now also U?.17 (D5)
- net VCC: now also U?.14 (VCC), U?.14 (VCC), U?.16 (VCC), U?.28 (VCC), U?.28 (VCC), U?.6 (E3)
- net at U?.10 (A0), U?.10 (A0), U?.2 (O0): now also U?.10 (A0), U?.10 (A0)
- net ALU_CARRY_IN: now reaches U?.11 (D0)
- net ALU_MODE: now reaches U?.12 (D1)
- net ALU_FUNCTION_SEL_0: now reaches U?.13 (D2)
- net ALU_FUNCTION_SEL_1: now reaches U?.15 (D3)
- net ALU_FUNCTION_SEL_2: now reaches U?.16 (D4)
- net ALU_FUNCTION_SEL_3: now reaches U?.17 (D5)
- net ALU_IN_AL_CLK: now reaches U?.18 (D6)
- net ALU_IN_AH_CLK: now reaches U?.19 (D7)
- net at U?.19 (O7), U?.3 (A7), U?.3 (A7): now also U?.3 (A7), U?.3 (A7)
- net at U?.16 (O6), U?.4 (A6), U?.4 (A6): now also U?.4 (A6), U?.4 (A6)
- net at U?.15 (O5), U?.5 (A5), U?.5 (A5): now also U?.5 (A5), U?.5 (A5)
- net at U?.12 (O4), U?.6 (A4), U?.6 (A4): now also U?.6 (A4), U?.6 (A4)
- net at U?.7 (A3), U?.7 (A3), U?.9 (O3): now also U?.7 (A3), U?.7 (A3)
- net at U?.6 (O2), U?.8 (A2), U?.8 (A2): now also U?.8 (A2), U?.8 (A2)
- net at U?.5 (O1), U?.9 (A1), U?.9 (A1): now also U?.9 (A1), U?.9 (A1)
- net ALU_IN_BL_CLK: now reaches U?.11 (D0)
- net ALU_IN_BH_CLK: now reaches U?.12 (D1)
- net -SRAM_WE: now reaches U?.18 (D6)
- net DATABUS_SEL_0: now reaches U?.19 (D7)
- net DATABUS_SEL_0: now also U?.1 (A0)
- new net: U?.1, U?.11 (O4)
- new net: U?.1, U?.10 (O5)
- new net -CODEROM_OE: U?.15 (O0)
- new net -CUR_CHAN_OE: U?.16 (D4)
- new net -IPH_OE: U?.13 (O2)
- new net -IPL_OE: U?.12 (O3)
- new net -SRAM_OE: U?.14 (O1)
- new net DATABUS_SEL_1: U?.11 (D0), U?.2 (A1)
- new net DATABUS_SEL_2: U?.12 (D1), U?.3 (A2)
- new net SELECT_BYTE: U?.17 (D5)
- new net SRAM_RANGE_SEL_0: U?.13 (D2)
- new net SRAM_RANGE_SEL_1: U?.15 (D3)
- no-connect marks 0 -> 12
Other:
- note added: "uCode ROM #0"
- note added: "uCode ROM #1"
- note added: "uCode ROM #2"
- note added: "uCode ROM #3"
- moved on the sheet: U?

Commit message: SRAM sheet
Connections:
- net -CUR_CHAN_OE renamed -CURRENT_CHANNEL_OE
- net SELECT_BYTE renamed BYTE_SELECT
Changed lines of the file:
@@
 Sheet 8 8
 Title ""
-Date "8 aug 2016"
+Date "9 aug 2016"
 Rev ""
 Comp ""
@@
 	12550 8850 12550 8200
 Text GLabel 12950 9000 2    60   Output ~ 0
--CUR_CHAN_OE
+-CURRENT_CHANNEL_OE
 Text GLabel 12950 9150 2    60   Output ~ 0
-SELECT_BYTE
+BYTE_SELECT
 Wire Wire Line
 	12950 9000 12450 9000

Commit message: weekly workshop update
Parts:
- added U? (x2): 74LS161, ~, symbol 74LS161
Connections:
- net GND: now also U?.8 (GND), U?.8 (GND)
- net VCC: now also U?.16 (VCC), U?.16 (VCC)
- net at U?.1 (A15): now also U?.1 (A15), U?.1 (A15), U?.1 (A15), U?.11 (Q3)
- net at U?.2 (A12): now also U?.2 (A12), U?.2 (A12), U?.2 (A12), U?.14 (Q0)
- net at U?.21 (A10): now also U?.21 (A10), U?.21 (A10), U?.24 (A9), U?.13 (Q1)
- net at U?.23 (A11): now also U?.23 (A11), U?.23 (A11), U?.25 (A8), U?.14 (Q0)
- net at U?.24 (A9): now also U?.21 (A10), U?.24 (A9), U?.24 (A9), U?.12 (Q2)
- net at U?.25 (A8): now also U?.23 (A11), U?.25 (A8), U?.25 (A8), U?.11 (Q3)
- net at U?.26 (A13): now also U?.26 (A13), U?.26 (A13), U?.26 (A13), U?.13 (Q1)
- net at U?.27 (A14): now also U?.27 (A14), U?.27 (A14), U?.27 (A14), U?.12 (Q2)
- new net: U?.10 (Cet), U?.15 (Tc), U?.7 (Cep)
- new net +5V: U?.10 (Cet), U?.7 (Cep), U?.9 (~Pe), U?.9 (~Pe)
- new net -CYCLE_COUNTER_CLK: U?.2 (Cp), U?.2 (Cp)
- new net -CYCLE_COUNTER_RESET: U?.1 (~MR), U?.1 (~MR)
- no-connect marks 12 -> 21
Other:
- note added: "Cycle Counter\nHigh"
- note added: "Cycle Counter\nLow"
- moved on the sheet: U?, U?A

Commit message: palette selection and video output circuitry (Color DAC and Palette ROM)
Connections:
- net CODEBANK_CLK renamed RESOURCE_BANK_CLK
Changed lines of the file:
@@
 $Descr A2 23386 16535
 encoding utf-8
-Sheet 6 7
+Sheet 6 8
 Title ""
-Date "9 aug 2016"
+Date "10 aug 2016"
 Rev ""
 Comp ""
@@
 ALU_IN_BL_CLK
 Text GLabel 14950 10150 2    60   Output ~ 0
-CODEBANK_CLK
+RESOURCE_BANK_CLK
 Text GLabel 14950 10300 2    60   Output ~ 0
 IPL_CLK
