File: anotherworld/microcode.sch (KiCad schematic (older format))
At the start: 10 parts

Commit message: rescue (loading the project on a newer git-revision of kicad)
Parts:
- U?: symbol 74LS374 -> 74LS374-RESCUE-anotherworld
- U? (x2): symbol 74HC04 -> 74HC04-RESCUE-anotherworld
- U?: symbol 74LS138 -> 74LS138-RESCUE-anotherworld
- U? (x2): symbol 74LS161 -> 74LS161-RESCUE-anotherworld
Changed lines of the file:
@@
 EESchema Schematic File Version 2
-LIBS:power
-LIBS:device
-LIBS:transistors
-LIBS:conn
-LIBS:linear
-LIBS:regul
-LIBS:74xx
-LIBS:cmos4000
-LIBS:adc-dac
-LIBS:memory
-LIBS:xilinx
-LIBS:special
-LIBS:microcontrollers
-LIBS:dsp
-LIBS:microchip
-LIBS:analog_switches
-LIBS:motorola
-LIBS:texas
-LIBS:intel
-LIBS:audio
-LIBS:interface
-LIBS:digital-audio
-LIBS:philips
-LIBS:display
-LIBS:cypress
-LIBS:siliconi
-LIBS:opto
-LIBS:atmel
-LIBS:contrib
-LIBS:valves
+LIBS:anotherworld-rescue
 LIBS:27c801
 LIBS:o_ttl
 LIBS:jamma_connector
 LIBS:anotherworld-cache
-EELAYER 25 0
+EELAYER 26 0
 EELAYER END
 $Descr A2 23386 16535
@@
 $EndComp
 $Comp
-L 74LS374 U?
+L 74LS374-RESCUE-anotherworld U?
 U 1 1 57A7EB1A
 P 6700 6450
@@
 ALU_OUT_L
 $Comp
-L 74HC04 U?
+L 74HC04-RESCUE-anotherworld U?
 U 1 1 57A8AE99
 P 8350 13500
@@
 $EndComp
 $Comp
-L 74HC04 U?
+L 74HC04-RESCUE-anotherworld U?
 U 1 1 57A8AF2C
 P 7650 13700
@@
 NoConn ~ 9650 9650
 $Comp
-L 74LS138 U?
+L 74LS138-RESCUE-anotherworld U?
 U 1 1 57A8CB1F
 P 7200 12100
@@
 $EndComp
 $Comp
-L 74LS161 U?
+L 74LS161-RESCUE-anotherworld U?
 U 1 1 57AA2BDB
 P 9450 3600
@@
 $EndComp
 $Comp
-L 74LS161 U?
+L 74LS161-RESCUE-anotherworld U?
 U 1 1 57AA2C03
 P 8050 3600
