File: anotherworld/jamma.sch (KiCad schematic (older format))
At the start: 0 parts

Commit message: jamma connector and signals, 320x200 video signals, etc...
Parts:
- added JAMMA1: JAMMA_CONNECTOR, symbol JAMMA_CONNECTOR
Connections:
- new net +5V: JAMMA1.3 (+5VDC), JAMMA1.4 (+5VDC), JAMMA1.C (+5VDC), JAMMA1.D (+5VDC)
- new net +SPEAKER: JAMMA1.10 (+SPEAKER)
- new net -SPEAKER: JAMMA1.L (-SPEAKER)
- new net BLUE: JAMMA1.13 (VIDEO_BLUE)
- new net GND: JAMMA1.1 (GROUND), JAMMA1.2 (GROUND), JAMMA1.27 (GROUND), JAMMA1.28 (GROUND), JAMMA1.A (GROUND), JAMMA1.B (GROUND), JAMMA1.e (GROUND), JAMMA1.f (GROUND)
- new net GREEN: JAMMA1.N (VIDEO_GREEN)
- new net PLAYER_ACTION: JAMMA1.22 (PLAYER_#1_BUTTON_1), JAMMA1.23 (PLAYER_#1_BUTTON_2), JAMMA1.24 (PLAYER_#1_BUTTON_3)
- new net PLAYER_DOWN: JAMMA1.19 (PLAYER_#1_DOWN)
- new net PLAYER_LEFT: JAMMA1.20 (PLAYER_#1_LEFT)
- new net PLAYER_RIGHT: JAMMA1.21 (PLAYER_#1_RIGHT)
- new net PLAYER_START: JAMMA1.17 (PLAYER_#1_START)
- new net PLAYER_UP: JAMMA1.18 (PLAYER_#1_UP)
- new net RED: JAMMA1.12 (VIDEO_RED)
- new net VIDEO_GND: JAMMA1.14 (VIDEO_GROUND)
- new net VSYNC: JAMMA1.P (VIDEO_SYNC)
- no-connect marks 0 -> 20
Changed lines of the file:
@@
 LIBS:27c801
 LIBS:o_ttl
+LIBS:jamma_connector
 LIBS:anotherworld-cache
 EELAYER 27 0
@@
 Sheet 2 8
 Title ""
-Date "12 aug 2016"
+Date "16 aug 2016"
 Rev ""
 Comp ""
@@
 Comment4 ""
 $EndDescr
+Text GLabel 13300 7500 2    60   Input ~ 0
+RED
+Text GLabel 10100 7500 0    60   Input ~ 0
+GREEN
+Text GLabel 12950 7600 2    60   Input ~ 0
+BLUE
+Text GLabel 9700 7600 0    60   Input ~ 0
+VSYNC
+$Comp
+L +5V #PWR?
+U 1 1 57B2DE52
+P 9800 6450
+F 0 "#PWR?" H 9800 6540 20  0001 C CNN
+F 1 "+5V" H 9800 6540 30  0000 C CNN
+F 2 "" H 9800 6450 60  0000 C CNN
+F 3 "" H 9800 6450 60  0000 C CNN
+	1    9800 6450
+	1    0    0    -1
+$EndComp
+$Comp
+L JAMMA_CONNECTOR JAMMA1
+U 1 1 57B302FA
+P 11500 7750
+F 0 "JAMMA1" H 10700 9350 60  0000 C CNN
+F 1 "JAMMA_CONNECTOR" H 11550 6250 60  0000 C CNN
+F 2 "" H 11500 8500 60  0000 C CNN
+F 3 "" H 11500 8500 60  0000 C CNN
+	1    11500 7750
+	1    0    0    -1
+$EndComp
+Wire Wire Line
+	10250 6600 9800 6600
+Wire Wire Line
+	9800 6450 9800 6700
+Wire Wire Line
+	9800 6700 10250 6700
+Connection ~ 9800 6600
+$Comp
+L +5V #PWR?
+U 1 1 57B3031F
+P 13200 6450
+F 0 "#PWR?" H 13200 6540 20  0001 C CNN
+F 1 "+5V" H 13200 6540 30  0000 C CNN
+F 2 "" H 13200 6450 60  0000 C CNN
+F 3 "" H 13200 6450 60  0000 C CNN
+	1    13200 6450
+	-1   0    0    -1
+$EndComp
+Wire Wire Line
+	12750 6600 13200 6600
+Wire Wire Line
+	13200 6450 13200 6700
+Wire Wire Line
+	13200 6700 12750 6700
+Connection ~ 13200 6600
+Wire Wire Line
+	13300 7500 12750 7500
+Wire Wire Line
+	12950 7600 12750 7600
+Wire Wire Line
+	9700 7600 10250 7600
+Wire Wire Line
+	10250 7500 10100 7500
+$Comp
+L GND #PWR?
+U 1 1 57B3035A
+P 9950 6800
+F 0 "#PWR?" H 9950 6800 30  0001 C CNN
+F 1 "GND" H 9950 6730 30  0001 C CNN
+F 2 "" H 9950 6800 60  0000 C CNN
+F 3 "" H 9950 6800 60  0000 C CNN
+	1    9950 6800
+	1    0    0    -1
+$EndComp
+Wire Wire Line
+	9950 6400 9950 6800
+Wire Wire Line
+	9950 6400 10250 6400
+Wire Wire Line
+	10250 6500 9950 6500
+Connection ~ 9950 6500
+$Comp
+L GND #PWR?
+U 1 1 57B3039A
+P 13050 6800
+F 0 "#PWR?" H 13050 6800 30  0001 C CNN
+F 1 "GND" H 13050 6730 30  0001 C CNN
+F 2 "" H 13050 6800 60  0000 C CNN
+F 3 "" H 13050 6800 60  0000 C CNN
+	1    13050 6800
+	1    0    0    -1
+$EndComp
+Wire Wire Line
+	12750 6400 13050 6400
+Wire Wire Line
+	13050 6400 13050 6800
+Wire Wire Line
+	12750 6500 13050 6500
+Connection ~ 13050 6500
+NoConn ~ 12750 6800
+NoConn ~ 12750 6900
+NoConn ~ 10250 6800
+NoConn ~ 10250 6900
+NoConn ~ 10250 7100
+NoConn ~ 10250 7200
+NoConn ~ 12750 7200
+NoConn ~ 10250 7800
+NoConn ~ 10250 7900
+NoConn ~ 10250 8000
+NoConn ~ 10250 8100
+NoConn ~ 10250 8200
+NoConn ~ 10250 8300
+NoConn ~ 10250 8400
+NoConn ~ 10250 8500
+NoConn ~ 10250 8600
+NoConn ~ 10250 8700
+Wire Wire Line
+	12750 8500 12900 8500
+Wire Wire Line
+	12900 8500 12900 8700
+Wire Wire Line
+	12900 8700 12750 8700
+Wire Wire Line
+	12750 8600 13150 8600
+Connection ~ 12900 8600
+Text GLabel 13150 8600 2    60   Output ~ 0
+PLAYER_ACTION
+Text GLabel 13150 8400 2    60   Output ~ 0
+PLAYER_RIGHT
+Text GLabel 13950 8300 2    60   Output ~ 0
+PLAYER_LEFT
+Text GLabel 13150 8200 2    60   Output ~ 0
+PLAYER_DOWN
+Text GLabel 13950 8100 2    60   Output ~ 0
+PLAYER_UP
+Text GLabel 13150 8000 2    60   Output ~ 0
+PLAYER_START
+Wire Wire Line
+	12750 8400 13150 8400
+Wire Wire Line
+	13950 8300 12750 8300
+Wire Wire Line
+	13150 8200 12750 8200
+Wire Wire Line
+	13950 8100 12750 8100
+Wire Wire Line
+	13150 8000 12750 8000
+NoConn ~ 12750 7800
+Text GLabel 13250 7700 2    60   Input ~ 0
+VIDEO_GND
+Wire Wire Line
+	13250 7700 12750 7700
+Text GLabel 12950 7300 2    60   Input ~ 0
++SPEAKER
+Wire Wire Line
+	12950 7300 12750 7300
+Text GLabel 10100 7300 0    60   Input ~ 0
+-SPEAKER
+Wire Wire Line
+	10100 7300 10250 7300
+NoConn ~ 12750 7100
+NoConn ~ 12750 7900
+$Comp
+L GND #PWR?
+U 1 1 57B30AF8
+P 12850 9300
+F 0 "#PWR?" H 12850 9300 30  0001 C CNN
+F 1 "GND" H 12850 9230 30  0001 C CNN
+F 2 "" H 12850 9300 60  0000 C CNN
+F 3 "" H 12850 9300 60  0000 C CNN
+	1    12850 9300
+	1    0    0    -1
+$EndComp
+Wire Wire Line
+	12850 9300 12850 9000
+Wire Wire Line
+	12850 9000 12750 9000
+Wire Wire Line
+	12750 9100 12850 9100
+Connection ~ 12850 9100
+$Comp
+L GND #PWR?
+U 1 1 57B30B44
+P 10150 9300
+F 0 "#PWR?" H 10150 9300 30  0001 C CNN
+F 1 "GND" H 10150 9230 30  0001 C CNN
+F 2 "" H 10150 9300 60  0000 C CNN
+F 3 "" H 10150 9300 60  0000 C CNN
+	1    10150 9300
+	-1   0    0    -1
+$EndComp
+Wire Wire Line
+	10150 9300 10150 9000
+Wire Wire Line
+	10150 9000 10250 9000
+Wire Wire Line
+	10250 9100 10150 9100
+Connection ~ 10150 9100
 $EndSCHEMATC

Commit message: weekly CPU from scratch workshop update
Connections:
- net VSYNC renamed SYNC
Changed lines of the file:
@@
 Sheet 2 8
 Title ""
-Date "16 aug 2016"
+Date "17 aug 2016"
 Rev ""
 Comp ""
@@
 BLUE
 Text GLabel 9700 7600 0    60   Input ~ 0
-VSYNC
+SYNC
 $Comp
 L +5V #PWR?

Commit message: an old set of changes (probably done last month during the Garoa workshops)
Connections:
- no-connect marks 20 -> 21
Changed lines of the file:
@@
 LIBS:jamma_connector
 LIBS:anotherworld-cache
-EELAYER 27 0
+EELAYER 25 0
 EELAYER END
 $Descr A2 23386 16535
@@
 NoConn ~ 10250 7800
 NoConn ~ 10250 7900
-NoConn ~ 10250 8000
-NoConn ~ 10250 8100
-NoConn ~ 10250 8200
-NoConn ~ 10250 8300
-NoConn ~ 10250 8400
 NoConn ~ 10250 8500
-NoConn ~ 10250 8600
 NoConn ~ 10250 8700
 Wire Wire Line
@@
 $EndComp
 Wire Wire Line
-	12850 9300 12850 9000
+	12850 9000 12850 9300
 Wire Wire Line
 	12850 9000 12750 9000
@@
 $EndComp
 Wire Wire Line
-	10150 9300 10150 9000
+	10150 9000 10150 9300
 Wire Wire Line
 	10150 9000 10250 9000
@@
 	10250 9100 10150 9100
 Connection ~ 10150 9100
+NoConn ~ 10250 8600
+NoConn ~ 10250 8400
+NoConn ~ 10250 8300
+NoConn ~ 10250 8200
+NoConn ~ 10250 8100
+NoConn ~ 10250 8000
+NoConn ~ 10250 7700
 $EndSCHEMATC
