File: anotherworld/master_clock.sch (KiCad schematic (older format))
At the start: 0 parts

Commit message: jamma connector and signals, 320x200 video signals, etc...
Other:
- note added: "TO-DO:\n\n15.75MHz\n\nPIXEL_CLOCK"
- note added: "TO-DO:\n\n? MHz\n\nMASTER_CLOCK\n\n(CRYSTAL\nOSCILATOR)"
Changed lines of the file:
@@
 LIBS:27c801
 LIBS:o_ttl
+LIBS:jamma_connector
 LIBS:anotherworld-cache
 EELAYER 27 0
@@
 Sheet 3 8
 Title ""
-Date "12 aug 2016"
+Date "16 aug 2016"
 Rev ""
 Comp ""
@@
 Comment4 ""
 $EndDescr
+Text Notes 4050 1600 0    157  ~ 0
+TO-DO:\n\n15.75MHz\n\nPIXEL_CLOCK
+Wire Notes Line
+	3700 1050 3700 3400
+Wire Notes Line
+	3700 3400 5900 3400
+Wire Notes Line
+	5900 3400 5900 1050
+Wire Notes Line
+	5900 1050 3700 1050
+Text Notes 1400 1450 0    157  ~ 0
+TO-DO:\n\n? MHz\n\nMASTER_CLOCK\n\n(CRYSTAL\nOSCILATOR)
+Wire Notes Line
+	1100 1050 1100 3400
+Wire Notes Line
+	1100 3400 3300 3400
+Wire Notes Line
+	3300 3400 3300 1050
+Wire Notes Line
+	3300 1050 1100 1050
 $EndSCHEMATC

Commit message: an old set of changes (probably done last month during the Garoa workshops)
Changed lines of the file:
@@
 LIBS:jamma_connector
 LIBS:anotherworld-cache
-EELAYER 27 0
+EELAYER 25 0
 EELAYER END
 $Descr A2 23386 16535
@@
 Comment4 ""
 $EndDescr
-Text Notes 4050 1600 0    157  ~ 0
+Text Notes 3950 2700 0    157  ~ 0
 TO-DO:\n\n15.75MHz\n\nPIXEL_CLOCK
 Wire Notes Line
@@
 Wire Notes Line
 	5900 1050 3700 1050
-Text Notes 1400 1450 0    157  ~ 0
+Text Notes 1400 3150 0    157  ~ 0
 TO-DO:\n\n? MHz\n\nMASTER_CLOCK\n\n(CRYSTAL\nOSCILATOR)
 Wire Notes Line
