File: anotherworld/video_output.sch (KiCad schematic (older format))
At the start: 39 parts

Commit message: drafting the HSYNC/VSYNC signal generation circuitry (work in pogress)
Parts:
- added U? (x2): 74LS161, ~, symbol 74LS161
- added U? (x3): 74LS93, ~, symbol 74LS93
- added U? (x2): 74LS74, ~, symbol 74LS74
- added U? (x4): 7402, ~, symbol 7402
- added U? (x2): 74LS08, ~, symbol 74LS08
- added U? (x2): 74LS10, ~, symbol 74LS10
- added U?: 74LS86, ~, symbol 74LS86
- added U?: 74HC04, ~, symbol 74HC04
- added U? (x2): 74LS107, ~, symbol 74LS107
Connections:
- net labels added: -512H, -COMP_SYNC, -HBLANK, -HRESET, -HSYNC, -VRESET, -VSYNC, 128H, 128V, 16V, 1V, 256H, 256V, 2H, 2V, 32H, 32V, 4V, 512V, 64H, 64V, 8V, CLOCK, COMP_SYNC, HBLANK, P, VRESET
- net labels removed: HSYNC
- wire segments 223 -> 320
Other:
- note added: "HRESET"
- note removed: "TODO:\nVSync & HSync\nsignals"

Commit message: improving the video signals generator (wip)
Connections:
- net labels added: 16H, 1H, 4H, 512H, 8H, HRESET
- wire segments 320 -> 338
- no-connect marks 14 -> 15
Other:
- note removed: "HRESET"
- moved on the sheet: U?, U?A, U?B, U?D

Commit message: jamma connector and signals, 320x200 video signals, etc...
Parts:
- removed U? (x2): 74LS74, ~, symbol 74LS74
- removed U? (x2): 74LS10, ~, symbol 74LS10
- removed U?: 74LS107, ~, symbol 74LS107
- added U? (x9): 74LS08, ~, symbol 74LS08
- added U? (x4): 7402, ~, symbol 7402
Connections:
- net labels added: +5V, -256H, -VBLANK, 200V, 320H, 336H, HSYNC, PIXEL_CLOCK, VBLANK
- net labels removed: -512H, -VRESET, 512H, 512V, CLOCK, P
- wire segments 338 -> 420
- no-connect marks 15 -> 25
Other:
- note added: "?????"
- note added: "HRes = 320"
- note added: "HSyncEnd = 368"
- note added: "HSyncStart = 336"
- note added: "HTotal = 416"
- note added: "TO-DO:\n\nVIDEO\nSRAM"
- note added: "VRes = 200"
- note added: "VSyncEnd = 202"
- note added: "VSyncStart = 200"
- note added: "VTotal = 222"
- moved on the sheet: R?, U?, U?A, U?B, U?D

Commit message: weekly CPU from scratch workshop update
Parts:
- removed U?: 74LS08, ~, symbol 74LS08
- added U?: 74LS32, ~, symbol 74LS32
Connections:
- net GND: now also U?.7 (GND)
- net HBLANK: now also U?.1; no longer U?.22 (OE), U?.22 (OE)
- net VBLANK: now also U?.2
- net VCC: now also U?.14 (VCC)
- net 202V: now reaches U?.11, U?.3
- net 202V: now also U?.1
- new net: U?.22 (OE), U?.22 (OE), U?.3
Changed lines of the file:
@@
 Sheet 7 8
 Title ""
-Date "16 aug 2016"
+Date "17 aug 2016"
 Rev ""
 Comp ""
@@
 Text GLabel 17150 1550 0    60   Input ~ 0
 2V
-Text GLabel 9350 13100 0    60   Input ~ 0
+Text GLabel 8050 13000 0    60   Input ~ 0
 HBLANK
 $Comp
@@
 	20200 2600 20400 2600
 Wire Wire Line
-	18500 1650 18850 1650
+	18500 1650 18650 1650
+Wire Wire Line
+	18650 1650 18850 1650
 Connection ~ 20200 2600
 Connection ~ 20200 1750
@@
 Text GLabel 19550 3850 2    60   Output ~ 0
 VRESET
-Text Notes 16300 3400 0    118  ~ 0
+Text Notes 16550 3800 0    118  ~ 0
 VTotal = 222
 $Comp
@@
 	18100 4200 17800 4200
 Wire Wire Line
-	17950 4000 18100 4000
-Wire Wire Line
 	19300 4100 19450 4100
 Wire Wire Line
@@
 Text GLabel 17900 2700 0    60   Input ~ 0
 200V
-Text GLabel 16400 3600 0    60   Input ~ 0
-200V
-Wire Wire Line
-	17950 3700 17950 4000
+Text GLabel 17800 4000 0    60   Input ~ 0
+202V
 Wire Wire Line
 	17900 2700 18850 2700
@@
 	19450 5400 19450 5150
 Connection ~ 19450 5150
-$Comp
-L 74LS08 U?
-U 1 1 57B2AFD0
-P 17200 3700
-F 0 "U?" H 17200 3750 60  0000 C CNN
-F 1 "74LS08" H 17200 3650 60  0000 C CNN
-F 2 "~" H 17200 3700 60  0000 C CNN
-F 3 "~" H 17200 3700 60  0000 C CNN
-	1    17200 3700
-	1    0    0    -1
-$EndComp
-Wire Wire Line
-	17950 3700 17800 3700
-Text GLabel 16400 3800 0    60   Input ~ 0
-2V
-Wire Wire Line
-	16600 3800 16400 3800
-Wire Wire Line
-	16400 3600 16600 3600
 Text Notes 10900 7650 0    197  ~ 0
 ?????
@@
 Wire Notes Line
 	4350 11300 2150 11300
-Text GLabel 23950 3750 2    60   Output ~ 0
+Text GLabel 8050 13200 0    60   Input ~ 0
 VBLANK
-Text GLabel 23900 3550 2    60   Output ~ 0
-VSYNC
-$Comp
-L +5V #PWR?
-U 1 1 57B2DE43
-P 24100 3250
-F 0 "#PWR?" H 24100 3340 20  0001 C CNN
-F 1 "+5V" H 24100 3340 30  0000 C CNN
-F 2 "" H 24100 3250 60  0000 C CNN
-F 3 "" H 24100 3250 60  0000 C CNN
-	1    24100 3250
-	1    0    0    -1
-$EndComp
+Wire Wire Line
+	8150 13000 8050 13000
+Wire Wire Line
+	8050 13200 8150 13200
+$Comp
+L 74LS32 U?
+U 1 1 57B3BEE4
+P 8750 13100
+F 0 "U?" H 8750 13150 60  0000 C CNN
+F 1 "74LS32" H 8750 13050 60  0000 C CNN
+F 2 "~" H 8750 13100 60  0000 C CNN
+F 3 "~" H 8750 13100 60  0000 C CNN
+	1    8750 13100
+	1    0    0    -1
+$EndComp
+Text GLabel 18750 1450 2    60   Output ~ 0
+202V
+Wire Wire Line
+	18750 1450 18650 1450
+Wire Wire Line
+	18650 1450 18650 1650
+Connection ~ 18650 1650
+Wire Wire Line
+	18100 4000 17800 4000
 $EndSCHEMATC

Commit message: rescue (loading the project on a newer git-revision of kicad)
Parts:
- U?: symbol 74LS374 -> 74LS374-RESCUE-anotherworld
- U? (x2): symbol 74LS161 -> 74LS161-RESCUE-anotherworld
- U? (x3): symbol 74LS93 -> 74LS93-RESCUE-anotherworld
- U? (x8): symbol 7402 -> 7402-RESCUE-anotherworld
- U? (x10): symbol 74LS08 -> 74LS08-RESCUE-anotherworld
- U?: symbol 74LS86 -> 74LS86-RESCUE-anotherworld
- U?: symbol 74HC04 -> 74HC04-RESCUE-anotherworld
- U?: symbol 74LS107 -> 74LS107-RESCUE-anotherworld
- U?: symbol 74LS32 -> 74LS32-RESCUE-anotherworld
Changed lines of the file:
@@
 EESchema Schematic File Version 2
-LIBS:power
-LIBS:device
-LIBS:transistors
-LIBS:conn
-LIBS:linear
-LIBS:regul
-LIBS:74xx
-LIBS:cmos4000
-LIBS:adc-dac
-LIBS:memory
-LIBS:xilinx
-LIBS:special
-LIBS:microcontrollers
-LIBS:dsp
-LIBS:microchip
-LIBS:analog_switches
-LIBS:motorola
-LIBS:texas
-LIBS:intel
-LIBS:audio
-LIBS:interface
-LIBS:digital-audio
-LIBS:philips
-LIBS:display
-LIBS:cypress
-LIBS:siliconi
-LIBS:opto
-LIBS:atmel
-LIBS:contrib
-LIBS:valves
+LIBS:anotherworld-rescue
 LIBS:27c801
 LIBS:o_ttl
 LIBS:jamma_connector
 LIBS:anotherworld-cache
-EELAYER 25 0
+EELAYER 26 0
 EELAYER END
 $Descr A2 23386 16535
@@
 RESOURCE_BANK_0
 $Comp
-L 74LS374 U?
+L 74LS374-RESCUE-anotherworld U?
 U 1 1 57AAD507
 P 8200 11400
@@
 DATA_5
 $Comp
-L 74LS161 U?
+L 74LS161-RESCUE-anotherworld U?
 U 1 1 57ACD7A3
 P 3300 3100
@@
 $EndComp
 $Comp
-L 74LS161 U?
+L 74LS161-RESCUE-anotherworld U?
 U 1 1 57ACD7B0
 P 5050 3100
@@
 $EndComp
 $Comp
-L 74LS93 U?
+L 74LS93-RESCUE-anotherworld U?
 U 1 1 57ACD7D2
 P 4000 6250
@@
 $EndComp
 $Comp
-L 74LS93 U?
+L 74LS93-RESCUE-anotherworld U?
 U 1 1 57ACD7FA
 P 5200 6250
@@
 $EndComp
 $Comp
-L 74LS93 U?
+L 74LS93-RESCUE-anotherworld U?
 U 1 1 57ACD800
 P 6400 6250
@@
 NoConn ~ 6400 7000
 $Comp
-L 7402 U?
+L 7402-RESCUE-anotherworld U?
 U 4 1 57ACED17
 P 19450 1750
+AR Path="/57ACED17" Ref="U?"  Part="4"
+AR Path="/57AAB07E/57ACED17" Ref="U?"  Part="4"
 F 0 "U?" H 19450 1800 60  0000 C CNN
 F 1 "7402" H 19500 1700 60  0000 C CNN
@@
 $EndComp
 $Comp
-L 7402 U?
+L 7402-RESCUE-anotherworld U?
 U 1 1 57ACED24
 P 19450 2600
+AR Path="/57ACED24" Ref="U?"  Part="1"
+AR Path="/57AAB07E/57ACED24" Ref="U?"  Part="1"
 F 0 "U?" H 19450 2650 60  0000 C CNN
 F 1 "7402" H 19500 2550 60  0000 C CNN
@@
 128V
 $Comp
-L 74LS08 U?
+L 74LS08-RESCUE-anotherworld U?
 U 2 1 57AD00E1
 P 18700 5150
+AR Path="/57AD00E1" Ref="U?"  Part="2"
+AR Path="/57AAB07E/57AD00E1" Ref="U?"  Part="2"
 F 0 "U?" H 18700 5200 60  0000 C CNN
 F 1 "74LS08" H 18700 5100 60  0000 C CNN
@@
 128H
 $Comp
-L 74LS08 U?
+L 74LS08-RESCUE-anotherworld U?
 U 1 1 57AD41D2
 P 11300 3000
+AR Path="/57AD41D2" Ref="U?"  Part="1"
+AR Path="/57AAB07E/57AD41D2" Ref="U?"  Part="1"
 F 0 "U?" H 11300 3050 60  0000 C CNN
 F 1 "74LS08" H 11300 2950 60  0000 C CNN
@@
 16H
 $Comp
-L 7402 U?
+L 7402-RESCUE-anotherworld U?
 U 1 1 57AD5942
 P 12550 1200
+AR Path="/57AD5942" Ref="U?"  Part="1"
+AR Path="/57AAB07E/57AD5942" Ref="U?"  Part="1"
 F 0 "U?" H 12550 1250 60  0000 C CNN
 F 1 "7402" H 12600 1150 60  0000 C CNN
@@
 $EndComp
 $Comp
-L 7402 U?
+L 7402-RESCUE-anotherworld U?
 U 1 1 57AD5948
 P 12550 2050
+AR Path="/57AD5948" Ref="U?"  Part="1"
+AR Path="/57AAB07E/57AD5948" Ref="U?"  Part="1"
 F 0 "U?" H 12550 2100 60  0000 C CNN
 F 1 "7402" H 12600 2000 60  0000 C CNN
@@
 -HRESET
 $Comp
-L 74LS86 U?
+L 74LS86-RESCUE-anotherworld U?
 U 2 1 57AD6F39
 P 11300 7950
+AR Path="/57AD6F39" Ref="U?"  Part="2"
+AR Path="/57AAB07E/57AD6F39" Ref="U?"  Part="2"
 F 0 "U?" H 11350 8000 50  0000 C CNN
 F 1 "74LS86" H 11350 7900 40  0000 C CNN
@@
 -COMP_SYNC
 $Comp
-L 74HC04 U?
+L 74HC04-RESCUE-anotherworld U?
 U 1 1 57AD729C
 P 12650 8250
+AR Path="/57AD729C" Ref="U?"  Part="1"
+AR Path="/57AAB07E/57AD729C" Ref="U?"  Part="1"
 F 0 "U?" H 12800 8350 40  0000 C CNN
 F 1 "74HC04" H 12850 8150 40  0000 C CNN
@@
 VSYNC
 $Comp
-L 74LS107 U?
+L 74LS107-RESCUE-anotherworld U?
 U 1 1 57AD7A10
 P 6800 3100
+AR Path="/57AD7A10" Ref="U?"  Part="1"
+AR Path="/57AAB07E/57AD7A10" Ref="U?"  Part="1"
 F 0 "U?" H 6800 3200 60  0000 C CNN
 F 1 "74LS107" H 6800 3000 60  0000 C CNN
@@
 NoConn ~ 5050 2400
 $Comp
-L 74LS08 U?
+L 74LS08-RESCUE-anotherworld U?
 U 1 1 57B20A82
 P 11150 2150
+AR Path="/57B20A82" Ref="U?"  Part="1"
+AR Path="/57AAB07E/57B20A82" Ref="U?"  Part="1"
 F 0 "U?" H 11150 2200 60  0000 C CNN
 F 1 "74LS08" H 11150 2100 60  0000 C CNN
@@
 HTotal = 416
 $Comp
-L 74LS08 U?
+L 74LS08-RESCUE-anotherworld U?
 U 1 1 57B20DB7
 P 12700 2900
+AR Path="/57B20DB7" Ref="U?"  Part="1"
+AR Path="/57AAB07E/57B20DB7" Ref="U?"  Part="1"
 F 0 "U?" H 12700 2950 60  0000 C CNN
 F 1 "74LS08" H 12700 2850 60  0000 C CNN
@@
 256H
 $Comp
-L 74LS08 U?
+L 74LS08-RESCUE-anotherworld U?
 U 1 1 57B21509
 P 17200 5250
+AR Path="/57B21509" Ref="U?"  Part="1"
+AR Path="/57AAB07E/57B21509" Ref="U?"  Part="1"
 F 0 "U?" H 17200 5300 60  0000 C CNN
 F 1 "74LS08" H 17200 5200 60  0000 C CNN
@@
 8V
 $Comp
-L 74LS08 U?
+L 74LS08-RESCUE-anotherworld U?
 U 1 1 57B21878
 P 17900 1650
+AR Path="/57B21878" Ref="U?"  Part="1"
+AR Path="/57AAB07E/57B21878" Ref="U?"  Part="1"
 F 0 "U?" H 17900 1700 60  0000 C CNN
 F 1 "74LS08" H 17900 1600 60  0000 C CNN
@@
 Connection ~ 9700 13100
 $Comp
-L 7402 U?
+L 7402-RESCUE-anotherworld U?
 U 1 1 57B22C92
 P 20250 4200
+AR Path="/57B22C92" Ref="U?"  Part="1"
+AR Path="/57AAB07E/57B22C92" Ref="U?"  Part="1"
 F 0 "U?" H 20250 4250 60  0000 C CNN
 F 1 "7402" H 20300 4150 60  0000 C CNN
@@
 $EndComp
 $Comp
-L 7402 U?
+L 7402-RESCUE-anotherworld U?
 U 1 1 57B22C98
 P 20250 5050
+AR Path="/57B22C98" Ref="U?"  Part="1"
+AR Path="/57AAB07E/57B22C98" Ref="U?"  Part="1"
 F 0 "U?" H 20250 5100 60  0000 C CNN
 F 1 "7402" H 20300 5000 60  0000 C CNN
@@
 16H
 $Comp
-L 74LS08 U?
+L 74LS08-RESCUE-anotherworld U?
 U 1 1 57B2320B
 P 17200 4200
+AR Path="/57B2320B" Ref="U?"  Part="1"
+AR Path="/57AAB07E/57B2320B" Ref="U?"  Part="1"
 F 0 "U?" H 17200 4250 60  0000 C CNN
 F 1 "74LS08" H 17200 4150 60  0000 C CNN
@@
 VTotal = 222
 $Comp
-L 74LS08 U?
+L 74LS08-RESCUE-anotherworld U?
 U 1 1 57B23213
 P 18700 4100
+AR Path="/57B23213" Ref="U?"  Part="1"
+AR Path="/57AAB07E/57B23213" Ref="U?"  Part="1"
 F 0 "U?" H 18700 4150 60  0000 C CNN
 F 1 "74LS08" H 18700 4050 60  0000 C CNN
@@
 	7650 3350 7450 3350
 $Comp
-L 7402 U?
+L 7402-RESCUE-anotherworld U?
 U 1 1 57B29E2D
 P 12700 4450
+AR Path="/57B29E2D" Ref="U?"  Part="1"
+AR Path="/57AAB07E/57B29E2D" Ref="U?"  Part="1"
 F 0 "U?" H 12700 4500 60  0000 C CNN
 F 1 "7402" H 12750 4400 60  0000 C CNN
@@
 $EndComp
 $Comp
-L 7402 U?
+L 7402-RESCUE-anotherworld U?
 U 1 1 57B29E33
 P 12700 5300
+AR Path="/57B29E33" Ref="U?"  Part="1"
+AR Path="/57AAB07E/57B29E33" Ref="U?"  Part="1"
 F 0 "U?" H 12700 5350 60  0000 C CNN
 F 1 "7402" H 12750 5250 60  0000 C CNN
@@
 336H
 $Comp
-L 74LS08 U?
+L 74LS08-RESCUE-anotherworld U?
 U 1 1 57B29E67
 P 11300 4350
+AR Path="/57B29E67" Ref="U?"  Part="1"
+AR Path="/57AAB07E/57B29E67" Ref="U?"  Part="1"
 F 0 "U?" H 11300 4400 60  0000 C CNN
 F 1 "74LS08" H 11300 4300 60  0000 C CNN
@@
 	10500 4450 10700 4450
 $Comp
-L 74LS08 U?
+L 74LS08-RESCUE-anotherworld U?
 U 1 1 57B2A01A
 P 11300 5400
+AR Path="/57B2A01A" Ref="U?"  Part="1"
+AR Path="/57AAB07E/57B2A01A" Ref="U?"  Part="1"
 F 0 "U?" H 11300 5450 60  0000 C CNN
 F 1 "74LS08" H 11300 5350 60  0000 C CNN
@@
 	8050 13200 8150 13200
 $Comp
-L 74LS32 U?
+L 74LS32-RESCUE-anotherworld U?
 U 1 1 57B3BEE4
 P 8750 13100
