File: anotherworld/video_output.sch (KiCad schematic (older format))
At the start: 66 parts

Commit message: update some file changes that were sitting on my local copy of the repo.
I sincerely have no idea what that was. Maybe just some caching of data from a previously opened session.
Parts:
- removed U? (x2): 74LS161, ~, symbol anotherworld-rescue:74LS161-RESCUE-anotherworld
- removed U? (x3): 74LS93, ~, symbol anotherworld-rescue:74LS93-RESCUE-anotherworld
- removed U?: 74LS107, ~, symbol anotherworld-rescue:74LS107-RESCUE-anotherworld
- added U? (x6): 74LS393, symbol o_ttl:74LS393
Connections:
- net labels added: 512H
- net labels removed: -256H, -HRESET
- wire segments 421 -> 377
- no-connect marks 25 -> 17
